File: PCB/board_eagle/nixie_schema.brd (EAGLE design)
At the start: 200 x 160 mm, 86 parts, among them IC1 LM2672M, Q1 BC856B, Q2 IRF740S

Commit message: Added cheaper 3V3 PSU
Parts:
- removed C7, C8: 100u, rcl:140CLH-0810
- removed D5: MBRS130LT3, diode:SMB
- removed D6: (no value), SparkFun-LED:LED-0603
- removed IC1: LM2672M, v-reg-3:SO08
- removed L2: 4.7u, rcl:CEP125
- removed R8: 1.33k, resistor:R0603
- added D3: (no value), diode:SOD123
- added R32: 5.6k, resistor:R0603
- added U$5: MC34063, MC34063:SOIC08
- C11: value 680p -> 10n
- C4: value 100u -> 270p; device rcl:140CLH-0810 -> eagle-ltspice:C0805
- C5: value 0.01 -> 100u; device Murata_By_element14_Batch_1:CAPC3216X180N -> rcl:153CLV-1014
- C6: value 0.022 -> 100u; device Murata_By_element14_Batch_1:CAPC3216X180N -> rcl:153CLV-1014
- L1: device rcl:CEP125 -> nixe_cmp:INDUCTOR_PACKAGE
- R10: value (none) -> 3.3k
- R22, R23: value (none) -> 0.5R
- R9: value 2,37K -> 0.5R; device resistor:R0603 -> eagle-ltspice:R1210
- moved C6 557.0 mm to (-133.3, -488.9)
- moved C5 530.5 mm to (-133.3, -463.6)
- moved R10 527.3 mm to (-143.5, -438.1)
- moved R9 501.6 mm to (-142.2, -424.2)
- moved L1 495.0 mm to (-135.9, -448.3)
- moved C4 492.5 mm to (-142.2, -431.8)
Connections:
- removed net N$100: R18.2
- removed net N$101: R17.2
- removed net N$102: R16.2
- removed net N$15: D6.A, R10.2
- removed net N$93: R15.2
- removed net N$94: R20.2
- removed net N$99: R19.2
- new net N$103: R10.1, R32.2, U$5.5
- net +3V3: now also C5.+, C6.+, L1.P$2, R32.1; no longer C8.+, L2.2, R10.1
- net GND: now also C4.2, C5.-, C6.-, D3.A, R10.2, U$5.4; no longer C4.-, C6.1, C7.-, C8.-, D5.A, D6.C, IC1.6, R8.2
- net HV_IN+: now also R15.2, R16.2, R17.2, R18.2, R19.2, R20.2; no longer R17.1, R18.1, SV3.11, SV3.12, SV4.11, SV4.12
- net N$11: now also R17.1, SV3.11, SV3.12; no longer C5.1, IC1.1
- net N$12: now also C4.1, U$5.3; no longer C5.2, D5.C, IC1.8, L1.1, R9.1
- net N$13: now also D3.C, L1.P$1, U$5.2; no longer C7.+, L1.2, L2.1
- net N$5: now also R9.2, U$5.1, U$5.7, U$5.8; no longer C6.2, IC1.2
- net N$8: now also R18.1, SV4.11, SV4.12; no longer IC1.4, R8.1, R9.2
- net VCC: now also R9.1, U$5.6; no longer C4.+, IC1.7

Commit message: Added optional RTC module and cleaned up the schematic
Parts:
- removed J2: (no value), SparkFun-Connectors:1X06_NO_SILK
- added C14, C17, C18, C7, C8: 100n, rcl:C0805
- added C15, C16: (no value), rcl:C0805
- added G1: CR2032H, battery:CR2032H
- added R8: (no value), resistor:R0603
- added S6: TAC_SWITCHSMD, SparkFun-Retired:TACTILE-SWITCH-SMD
- added U2: MC7940N, nixe_cmp:SOIC8-N_MC
- added Y1: (no value), crystal:SM49
- C1, C3: device rcl:140CLH-0810 -> rcl:C0805
- C10, C11, C4: device eagle-ltspice:C0805 -> rcl:C0805
- C9: value (none) -> 10u
- R1, R2, R3, R4, R5, R6: value 2.21K -> 2.2k
- R28, R29, R30, R7: value 2.21K -> 2.2K
- moved C5 391.0 mm to (-90.2, -74.9)
- moved C6 391.0 mm to (-90.2, -100.3)
- moved D3 391.0 mm to (-97.8, -91.4)
- moved L1 391.0 mm to (-92.7, -59.7)
- moved R10 391.0 mm to (-100.3, -49.5)
- moved R15 391.0 mm to (-100.3, 26.7)
- moved R17 391.0 mm to (-100.3, 16.5)
- moved R18 391.0 mm to (-100.3, 11.4)
- moved R19 391.0 mm to (-100.3, 6.35)
- moved R20 391.0 mm to (-100.3, 1.27)
- moved R32 391.0 mm to (-100.3, -85.1)
- moved R9 391.0 mm to (-99.1, -35.6)
- moved S1 391.0 mm to (-69.8, 31.8)
- moved U1 391.0 mm to (-88.9, 44.5)
- moved R16 391.0 mm to (-100.3, 21.6)
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Connections:
- new net N$100: C15.1, U2.2, Y1.2
- new net N$15: JP1.1, R13.2, S6.1, S6.2, U1.GPIO0
- new net N$99: C16.1, U2.1, Y1.1
- net +3V3: now also C17.1, C18.1, R28.2, R29.2, R30.2, R7.2, R8.1, U2.8; no longer J2.1, S2.3, S3.3, S4.3, S5.3
- net BUTTON1: now also J3.5, R7.1, S2.3, S2.4; no longer J2.2, J3.2, R30.2, S5.1, S5.2
- net BUTTON2: now also J3.4, R28.1, R8.2, S3.3, S3.4; no longer J2.3, J3.3, R29.2, S4.1, S4.2
- net BUTTON3: now also J3.3, R29.1, S4.3, S4.4, U2.6; no longer J2.4, J3.4, R28.2, S3.1, S3.2
- net BUTTON4: now also J3.2, R30.1, S5.3, S5.4, U2.5; no longer J2.5, J3.5, R7.2, S2.1, S2.2
- net GND: now also C15.2, C16.2, C17.2, C18.2, C7.2, G1.-, S1.1, S2.1, S2.2, S3.1, S3.2, S4.1, S4.2, S5.1, S5.2, S6.3, S6.4, U2.4; no longer C1.-, C10.2, C11.2, C3.-, C4.2, J2.6, R28.1, R29.1, R30.1, R7.1
- net N$12: no longer C4.1
- net N$14: now also S1.3
- net N$22: now also G1.+, U2.3; no longer JP1.1, R13.2, U1.GPIO0
- net N$74: no longer C10.1
- net N$96: no longer C11.1
- net VCC: no longer C1.+, C3.+
