File: PCB/board_eagle/nixie_schema.sch (EAGLE design)
At the start: 103 parts, among them J2 RTC_CONSMD, J4 RTC_CONTHT, P1 100k, Q1 BC856B, Q2 IRF740S, T1 PHOTO_TRANS, U2 MC7940N, Y1 ECS-.327-7-34B

Commit message: Top board touting complete
Connections:
- new net N$31: N2.7, SV8.4
- new net N$32: N2.8, SV8.6
- new net N$33: N2.9, SV8.8
- new net N$34: N2.0, SV8.10
- new net N$35: N3.RHDP, SV9.11
- new net N$36: N3.6, SV9.2
- new net N$37: N3.7, SV9.4
- new net N$38: N2.5, SV8.1
- new net N$39: N2.4, SV8.3
- new net N$40: N2.3, SV8.5
- new net N$41: N2.2, SV8.7
- new net N$42: N2.1, SV8.9
- new net N$43: N3.8, SV9.6
- new net N$44: N3.9, SV9.8
- new net N$46: N3.0, SV9.10
- new net N$47: N4.RHDP, SV10.11
- new net N$48: N4.6, SV10.2
- new net N$49: N3.5, SV9.1
- new net N$50: N3.4, SV9.3
- new net N$51: N3.3, SV9.5
- new net N$52: N3.2, SV9.7
- new net N$53: N3.1, SV9.9
- new net N$54: N4.7, SV10.4
- new net N$55: N4.8, SV10.6
- new net N$56: N4.9, SV10.8
- new net N$57: N4.0, SV10.10
- new net N$58: N5.RHDP, SV11.11
- new net N$59: N4.5, SV10.1
- new net N$60: N4.4, SV10.3
- new net N$61: N4.3, SV10.5
- new net N$62: N4.2, SV10.7
- new net N$63: N4.1, SV10.9
- new net N$64: N5.6, SV11.2
- new net N$65: N5.7, SV11.4
- new net N$66: N5.8, SV11.6
- new net N$67: N5.9, SV11.8
- new net N$68: N5.0, SV11.10
- new net N$69: N5.5, SV11.1
- new net N$70: N5.4, SV11.3
- new net N$71: N5.3, SV11.5
- new net N$72: N5.2, SV11.7
- new net N$73: N5.1, SV11.9
- new net N$75: N6.RHDP, SV12.11
- new net N$76: N6.6, SV12.2
- new net N$77: N6.7, SV12.4
- new net N$78: N6.8, SV12.6
- new net N$79: N6.9, SV12.8
- new net N$80: N6.5, SV12.1
- new net N$81: N6.4, SV12.3
- new net N$82: N6.3, SV12.5
- new net N$83: N6.2, SV12.7
- new net N$84: N6.1, SV12.9
- new net N$86: N6.0, SV12.10
- net HV_HA_1: now also SV1.9, U$1.HV6; no longer SV1.8, U$1.HV2
- net HV_HA_2: now also SV1.7, U$1.HV7; no longer SV1.6, U$1.HV3
- net HV_HA_3: now also SV1.5, U$1.HV8; no longer SV1.4, U$1.HV4
- net HV_HA_4: now also SV1.3, U$1.HV9; no longer SV1.2, U$1.HV5
- net HV_HA_5: now also SV1.1, U$1.HV10; no longer SV1.9, U$1.HV6
- net HV_HA_6: now also SV1.2, U$1.HV5; no longer SV1.7, U$1.HV7
- net HV_HA_7: now also SV1.4, U$1.HV4; no longer SV1.5, U$1.HV8
- net HV_HA_8: now also SV1.6, U$1.HV3; no longer SV1.3, U$1.HV9
- net HV_HA_9: now also SV1.8, U$1.HV2; no longer SV1.1, U$1.HV10
- net HV_HB_1: now also SV2.9, U$1.HV16; no longer SV2.8, U$1.HV19
- net HV_HB_2: now also SV2.7, U$1.HV15; no longer SV2.6, U$1.HV20
- net HV_HB_3: now also SV2.5, U$1.HV14; no longer SV2.4, U$1.HV21
- net HV_HB_4: now also SV2.3, U$1.HV13; no longer SV2.2, U$1.HV22
- net HV_HB_5: now also SV2.1, U$1.HV12; no longer SV2.9, U$1.HV16
- net HV_HB_6: now also SV2.2, U$1.HV22; no longer SV2.7, U$1.HV15
- net HV_HB_7: now also SV2.4, U$1.HV21; no longer SV2.5, U$1.HV14
- net HV_HB_8: now also SV2.6, U$1.HV20; no longer SV2.3, U$1.HV13
- net HV_HB_9: now also SV2.8, U$1.HV19; no longer SV2.1, U$1.HV12
- net HV_MA_1: now also SV3.9, U$1.HV28; no longer SV3.8, U$1.HV26
- net HV_MA_2: now also SV3.7, U$1.HV29; no longer SV3.6, U$1.HV25
- net HV_MA_3: now also SV3.5, U$1.HV30; no longer SV3.4, U$1.HV24
- net HV_MA_4: now also SV3.3, U$1.HV31; no longer SV3.2, U$1.HV23
- net HV_MA_5: now also SV3.1, U$1.HV32; no longer SV3.9, U$1.HV28
- net HV_MA_6: now also SV3.2, U$1.HV23; no longer SV3.7, U$1.HV29
- net HV_MA_7: now also SV3.4, U$1.HV24; no longer SV3.5, U$1.HV30
- net HV_MA_8: now also SV3.6, U$1.HV25; no longer SV3.3, U$1.HV31
- net HV_MA_9: now also SV3.8, U$1.HV26; no longer SV3.1, U$1.HV32
- net HV_MB_1: now also SV4.9, U$2.HV7; no longer SV4.8, U$2.HV4
- net HV_MB_2: now also SV4.7, U$2.HV8; no longer SV4.6, U$2.HV3
- net HV_MB_3: now also SV4.5, U$2.HV9; no longer SV4.4, U$2.HV2
- net HV_MB_4: now also SV4.3, U$2.HV10; no longer SV4.2, U$2.HV1
- net HV_MB_5: now also SV4.1, U$2.HV11; no longer SV4.9, U$2.HV7
- net HV_MB_6: now also SV4.2, U$2.HV1; no longer SV4.7, U$2.HV8
- net HV_MB_7: now also SV4.4, U$2.HV2; no longer SV4.5, U$2.HV9
- net HV_MB_8: now also SV4.6, U$2.HV3; no longer SV4.3, U$2.HV10
- net HV_MB_9: now also SV4.8, U$2.HV4; no longer SV4.1, U$2.HV11
- net HV_SA_1: now also SV5.9, U$2.HV17; no longer SV5.8, U$2.HV19
- net HV_SA_2: now also SV5.7, U$2.HV16; no longer SV5.6, U$2.HV20
- net HV_SA_3: now also SV5.5, U$2.HV15; no longer SV5.4, U$2.HV21
- net HV_SA_4: now also SV5.3, U$2.HV14; no longer SV5.2, U$2.HV22
- net HV_SA_5: now also SV5.1, U$2.HV13; no longer SV5.9, U$2.HV17
- net HV_SA_6: now also SV5.2, U$2.HV22; no longer SV5.7, U$2.HV16
- net HV_SA_7: now also SV5.4, U$2.HV21; no longer SV5.5, U$2.HV15
- net HV_SA_8: now also SV5.6, U$2.HV20; no longer SV5.3, U$2.HV14
- net HV_SA_9: now also SV5.8, U$2.HV19; no longer SV5.1, U$2.HV13
- net HV_SB_1: now also SV6.9, U$2.HV32; no longer SV6.8, U$2.HV26
- net HV_SB_2: now also SV6.7, U$2.HV31; no longer SV6.6, U$2.HV25
- net HV_SB_3: now also SV6.5, U$2.HV30; no longer SV6.4, U$2.HV24
- net HV_SB_4: now also SV6.3, U$2.HV29; no longer SV6.2, U$2.HV23
- net HV_SB_5: now also SV6.1, U$2.HV28; no longer SV6.9, U$2.HV32
- net HV_SB_6: now also SV6.2, U$2.HV23; no longer SV6.7, U$2.HV31
- net HV_SB_7: now also SV6.4, U$2.HV24; no longer SV6.5, U$2.HV30
- net HV_SB_8: now also SV6.6, U$2.HV25; no longer SV6.3, U$2.HV29
- net HV_SB_9: now also SV6.8, U$2.HV26; no longer SV6.1, U$2.HV28
- net N$1: now also SV8.11; no longer SV8.10
- net N$2: now also N1.6, SV7.2; no longer N1.0, SV7.8
- net N$23: now also N2.6, SV8.2; no longer N3.RHDP, SV9.10
- net N$24: now also N1.9, SV7.8; no longer N1.7, SV7.2
- net N$30: now also N1.RHDP; no longer N1.6
- net N$6: now also N1.7, SV7.4; no longer N1.9, SV7.6
- net N$7: now also SV7.6; no longer SV7.4
- net N$94: now also N1.0; no longer N1.RHDP

Commit message: Added some values to components in schematic
Parts:
- C15, C16: value (none) -> 6p
- D1: value (none) -> 1n4148
- R11, R12, R13, R14, R8: value (none) -> 10k
Other:
- note added: "C15;C16 = 2*Cload - 2*Cstray Cstray ~= 4pf https://blog.adafruit.com/2012/01/24/choosing-the-right-crystal-and-caps-for-your-design/"
Changed lines of the file:
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@@
 <part name="SV5" library="con-lstb" deviceset="MA06-2" device=""/>
 <part name="SV6" library="con-lstb" deviceset="MA06-2" device=""/>
-<part name="R11" library="resistor" deviceset="R-EU_" device="R0603"/>
-<part name="R12" library="resistor" deviceset="R-EU_" device="R0603"/>
-<part name="R13" library="resistor" deviceset="R-EU_" device="R0603"/>
-<part name="R14" library="resistor" deviceset="R-EU_" device="R0603"/>
+<part name="R11" library="resistor" deviceset="R-EU_" device="R0603" value="10k"/>
+<part name="R12" library="resistor" deviceset="R-EU_" device="R0603" value="10k"/>
+<part name="R13" library="resistor" deviceset="R-EU_" device="R0603" value="10k"/>
+<part name="R14" library="resistor" deviceset="R-EU_" device="R0603" value="10k"/>
 <part name="JP1" library="PatternAgents-JTAG" deviceset="JUMPER2" device=""/>
 <part name="U$14" library="PatternAgents-Beautify" deviceset="GND" device=""/>
@@
 <part name="R23" library="eagle-ltspice" deviceset="R" device="R1210" value="0.5R"/>
 <part name="SUPPLY7" library="SparkFun-PowerSymbols" deviceset="VCC" device=""/>
-<part name="D1" library="diode" deviceset="DIODE-" device="SOD123"/>
+<part name="D1" library="diode" deviceset="DIODE-" device="SOD123" value="1n4148"/>
 <part name="U$22" library="PatternAgents-Beautify" deviceset="GND" device=""/>
 <part name="U$23" library="PatternAgents-Beautify" deviceset="GND" device=""/>
@@
 <part name="U$11" library="PatternAgents-Beautify" deviceset="GND" device=""/>
 <part name="U$12" library="PatternAgents-Beautify" deviceset="GND" device=""/>
-<part name="C15" library="rcl" deviceset="C-EU" device="C0805"/>
-<part name="C16" library="rcl" deviceset="C-EU" device="C0805"/>
+<part name="C15" library="rcl" deviceset="C-EU" device="C0805" value="6p"/>
+<part name="C16" library="rcl" deviceset="C-EU" device="C0805" value="6p"/>
 <part name="GND14" library="supply1" deviceset="GND" device=""/>
 <part name="GND15" library="supply1" deviceset="GND" device=""/>
@@
 <part name="U$30" library="PatternAgents-Beautify" deviceset="GND" device=""/>
 <part name="U$31" library="PatternAgents-Beautify" deviceset="GND" device=""/>
-<part name="R8" library="resistor" deviceset="R-EU_" device="R0603"/>
+<part name="R8" library="resistor" deviceset="R-EU_" device="R0603" value="10k"/>
 <part name="Y1" library="nixe_cmp" deviceset="ECS-.327-7-34B" device="" value=""/>
 <part name="BAT1" library="nixe_cmp" deviceset="CR2032" device=""/>
@@
 Note:
    Populate either R8 or R28, not both</text>
+<text x="226.06" y="-38.1" size="1.778" layer="91">C15;C16 = 2*Cload - 2*Cstray
+Cstray ~= 4pf
+https://blog.adafruit.com/2012/01/24/choosing-the-right-crystal-and-caps-for-your-design/</text>
 </plain>
 <instances>
-<instance part="R11" gate="G$1" x="10.16" y="68.58" rot="R180"/>
-<instance part="R12" gate="G$1" x="10.16" y="63.5" rot="R180"/>
+<instance part="R11" gate="G$1" x="10.16" y="68.58" smashed="yes" rot="R180">
+<attribute name="NAME" x="8.89" y="72.1614" size="1.778" layer="95" rot="R180"/>
+<attribute name="VALUE" x="16.51" y="71.882" size="1.778" layer="96" rot="R180"/>
+</instance>
+<instance part="R12" gate="G$1" x="10.16" y="63.5" smashed="yes" rot="R180">
+<attribute name="NAME" x="8.89" y="62.0014" size="1.778" layer="95" rot="R180"/>
+<attribute name="VALUE" x="13.97" y="61.722" size="1.778" layer="96" rot="R180"/>
+</instance>
 <instance part="R13" gate="G$1" x="55.88" y="76.2" rot="R270"/>
 <instance part="R14" gate="G$1" x="66.04" y="53.34" rot="R180"/>
@@
 </sheet>
 </sheets>
+<errors>
+</errors>
 </schematic>
 </drawing>
